Commit message: add continuous set-points

File: src/gp4_moveit_config/config/motoman_gp4.ros2_control.xacro (robot description, xacro)
@@ -2,5 +2,5 @@
 <robot xmlns:xacro="http://www.ros.org/wiki/xacro">
     <xacro:macro name="motoman_gp4_ros2_control" params="name initial_positions_file use_fake_hardware:=false robot_ip:=192.168.1.33 controller_port:=50240">
-        <xacro:property name="initial_positions" value="${load_yaml(initial_positions_file)['initial_positions']}"/>
+        <xacro:property name="initial_positions" value="${xacro.load_yaml(initial_positions_file)['initial_positions']}"/>
         <ros2_control name="${name}" type="system">
             <hardware>

File: src/gp4_moveit_config/config/motoman_gp4.urdf.xacro (robot description, xacro)
@@ -7,5 +7,5 @@
           false = robot thật Yaskawa GP4 qua MotoROS2
     -->
-    <xacro:arg name="use_fake_hardware"       default="true" />
+    <xacro:arg name="use_fake_hardware"       default="false" />
     <xacro:arg name="robot_ip"                default="192.168.1.33" />
     <xacro:arg name="controller_port"         default="50240" />
